File: Signal_Board/Signal_Board.kicad_sch (KiCad schematic)
At the start: 17 parts, among them J1 Conn_01x02_Pin, J2 Conn_01x06_Pin, U1 74HC14, U2 LM317LZ, U3 4046

Commit message: Signal board version 0.0.2; updates in README
Parts:
- added TP1: GND, Connector_Pin:Pin_D1.0mm_L10.0mm, symbol Connector:TestPoint
- added TP2: 6 V, Connector_Pin:Pin_D1.0mm_L10.0mm, symbol Connector:TestPoint
- added TP3: Osc, Connector_Pin:Pin_D1.0mm_L10.0mm, symbol Connector:TestPoint
- added TP4: Sig, Connector_Pin:Pin_D1.0mm_L10.0mm, symbol Connector:TestPoint
- R1: renamed from R5; value 1k -> 240; footprint PCM_Resistor_THT_AKL:R_Axial_DIN0204_L3.6mm_D1.6mm_P5.08mm_Vertical -> PCM_Resistor_THT_AKL:R_Axial_DIN0204_L3.6mm_D1.6mm_P7.62mm_Horizontal
- R2: renamed from R6; value 3k6 -> 910; footprint PCM_Resistor_THT_AKL:R_Axial_DIN0204_L3.6mm_D1.6mm_P5.08mm_Vertical -> PCM_Resistor_THT_AKL:R_Axial_DIN0204_L3.6mm_D1.6mm_P7.62mm_Horizontal
- R3: renamed from R1; footprint PCM_Resistor_THT_AKL:R_Axial_DIN0204_L3.6mm_D1.6mm_P5.08mm_Vertical -> PCM_Resistor_THT_AKL:R_Axial_DIN0204_L3.6mm_D1.6mm_P7.62mm_Horizontal
- R4: renamed from R2; footprint PCM_Resistor_THT_AKL:R_Axial_DIN0204_L3.6mm_D1.6mm_P5.08mm_Vertical -> PCM_Resistor_THT_AKL:R_Axial_DIN0204_L3.6mm_D1.6mm_P7.62mm_Horizontal
- R5: renamed from R4; footprint PCM_Resistor_THT_AKL:R_Axial_DIN0204_L3.6mm_D1.6mm_P5.08mm_Vertical -> PCM_Resistor_THT_AKL:R_Axial_DIN0204_L3.6mm_D1.6mm_P7.62mm_Horizontal
- R6: renamed from R3; footprint PCM_Resistor_THT_AKL:R_Axial_DIN0204_L3.6mm_D1.6mm_P5.08mm_Vertical -> PCM_Resistor_THT_AKL:R_Axial_DIN0204_L3.6mm_D1.6mm_P7.62mm_Horizontal
- renumbered C4 to C1, C5 to C2, C2 to C3, C3 to C4, C1 to C5
Connections:
- net +6V: now also TP2.1
- net GND: now also TP1.1; no longer U1.10, U1.12, U1.4, U1.6, U1.8
- net OSC_Out: now also TP3.1
- net SIG_Out: now also TP4.1
- no-connect marks 5 -> 10
